File: FlightComputer V1/chips.kicad_sch (KiCad schematic)
At the start: 5 parts, among them U1 GYU-521, U3 W25Q64, U4 GY-BMP280, U5 Micro-SD-Card-Holder

Commit message: Added power circuitry
reset button, ADC for voltage detection, voltage regulator and switch for total power on and off. Screw terminal to interface between battery pack and PCB.
Connections:
- net Power renamed VCC
Changed lines of the file:
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@@
 		)
 	)
-	(global_label "Power"
+	(global_label "VCC"
 		(shape input)
 		(at 179.07 152.4 90)
@@
 		)
 		(property "Intersheetrefs" "${INTERSHEET_REFS}"
-			(at 179.07 143.7905 90)
+			(at 179.07 145.7862 90)
 			(effects
 				(font
