File: FlightComputer V1/untitled.kicad_sch (KiCad schematic)
At the start: 0 parts

Commit message: Added power circuitry
reset button, ADC for voltage detection, voltage regulator and switch for total power on and off. Screw terminal to interface between battery pack and PCB.
Parts:
- added D1: LED, symbol Device:LED
- added J1: Screw_Terminal_01x02, symbol Connector:Screw_Terminal_01x02
- added R5, R6, R7: R, symbol Device:R
- added SW1: SW_SPST, symbol Switch:SW_SPST
- added SW2: SW_Push, symbol Switch:SW_Push
- added U2: Voltage Regulator, symbol FlightComputerV1Parts:Voltage_Regulator_
Connections:
- new net: J1.1 (Pin_1), SW1.1 (A)
- new net: SW1.2 (B), U2. (VOUT)
- new net: D1.2 (A), R7.1
- new net ADC: R5.2, R6.1
- new net GND: D1.1 (K)
- new net GNDPWR: R6.2, SW2.1, U2. (VOUT)
- new net RUN: SW2.2
- new net VCC: R5.1, R7.2, U2. (VOUT)
